Commit message: Add files via upload

File: ackermann_vehicle_description/urdf/em_3905.urdf_V2.xacro (robot description, xacro)
@@ -30,4 +30,5 @@
 -->
 <robot name="em_3905" xmlns:xacro="http://www.ros.org/wiki/xacro">
+  <xacro:include filename="$(find ackermann_vehicle_description)/urdf/colors.xacro" />
   <!-- Degree-to-radian conversions -->
   <xacro:property name="degrees_45" value="0.785398163"/>
@@ -95,13 +96,4 @@
   <xacro:property name="servo_stall_torque" value="1.5649"/>
   <xacro:property name="servo_no_load_speed" value="4.5530"/>
-  <material name="battery_mat">
-    <color rgba="0 0 1 1"/>
-  </material>
-  <material name="chassis_mat">
-    <color rgba="0.5 0.5 0.5 1"/>
-  </material>
-  <material name="tire_mat">
-    <color rgba="0 0 0 1"/>
-  </material>
   <!-- Null inertial element. This is needed to make the model work with
        Gazebo. -->

Commit message: Add files via upload

File: ackermann_vehicle_description/urdf/em_3905.urdf_V2.xacro (robot description, xacro)
@@ -2,5 +2,5 @@
 <!-- MADE SOME CHANGES IN THE DIMENSIONS and MASS
 WHEEL MASS IS CORRECT, REST IS NOT -->
-<!-- Also added a camera and broke the materials to a different file -->
+<!-- rEMOVED THE BATTERIES -->
 <!-- em_3905.urdf.xacro
 This file defines a model of a Traxxas(R) E-Maxx(R) #3905 RC (Radio Controlled)
@@ -32,7 +32,4 @@
 <robot name="em_3905" xmlns:xacro="http://www.ros.org/wiki/xacro">
   <xacro:include filename="$(find ackermann_vehicle_description)/urdf/colors.xacro" />
-  <xacro:include filename="$(find ackermann_vehicle_description)/urdf/sensors.gazebo" />
-  <xacro:property name="cameraSize" value="0.05"/>
-  <xacro:property name="cameraMass" value="0.1"/>
   <!-- Degree-to-radian conversions -->
   <xacro:property name="degrees_45" value="0.785398163"/>
@@ -140,4 +137,5 @@
   </xacro:macro>
   <!-- Battery -->
+<!--
   <xacro:macro name="battery" params="prefix reflect">
     <joint name="chassis_to_${prefix}_battery" type="fixed">
@@ -181,4 +179,5 @@
     </gazebo>
   </xacro:macro>
+-->
   <!-- Shock absorber -->
   <xacro:macro name="shock"
@@ -343,6 +342,8 @@
   </joint>
   <!-- Batteries -->
+  <!--
   <xacro:battery prefix="left" reflect="1"/>
   <xacro:battery prefix="right" reflect="-1"/>
+  -->
   <!-- Wheels -->
   <xacro:front_wheel lr_prefix="left" fr_prefix="front"
@@ -354,31 +355,4 @@
   <xacro:rear_wheel lr_prefix="right" fr_prefix="rear"
                     lr_reflect="-1" fr_reflect="-1"/>
-  <link name="camera">
-    <collision>
-      <origin xyz="0 0 0" rpy="0 0 0"/>
-      <geometry>
-        <box size="${cameraSize} ${cameraSize} ${cameraSize}"/>
-      </geometry>
-    </collision>
-    <visual>
-      <origin xyz="0 0 0" rpy="0 0 0"/>
-      <geometry>
-        <box size="${cameraSize} ${cameraSize} ${cameraSize}"/>
-      </geometry>
-      <material name="green"/>
-    </visual>
-    <inertial>
-      <mass value="${cameraMass}" />
-      <origin xyz="0 0 0" rpy="0 0 0"/>
-      <box_inertia m="${cameraMass}" x="${cameraSize}" y="${cameraSize}" z="${cameraSize}" />
-      <inertia ixx="1e-6" ixy="0" ixz="0" iyy="1e-6" iyz="0" izz="1e-6" />
-    </inertial>
-  </link>
-  <joint name="camera_joint" type="fixed">
-    <axis xyz="0 1 0" />
-    <origin xyz=".2 0 1" rpy="0 0 0"/>
-    <parent link="chassis"/>
-    <child link="camera"/>
-  </joint>
   <gazebo>
     <plugin name="gazebo_ros_control" filename="libgazebo_ros_control.so"/>

File: ackermann_vehicle_description/urdf/em_3905.urdf_V4.xacro (robot description, xacro)
@@ -2,5 +2,5 @@
 <!-- MADE SOME CHANGES IN THE DIMENSIONS and MASS
 WHEEL MASS IS CORRECT, REST IS NOT -->
-<!-- Also added a camera, imu and broke the materials to a different file -->
+<!-- Also added a camera, imu, removed the batteries and broke the materials to a different file -->
 <!-- em_3905.urdf.xacro
 This file defines a model of a Traxxas(R) E-Maxx(R) #3905 RC (Radio Controlled)
@@ -139,46 +139,4 @@
     </inertial>
   </xacro:macro>
-  <!-- Battery -->
-  <xacro:macro name="battery" params="prefix reflect">
-    <joint name="chassis_to_${prefix}_battery" type="fixed">
-      <parent link="chassis"/>
-      <child link="${prefix}_battery_offset"/>
-      <origin xyz="${battery_x_offset - battery_length / 2}
-                   ${reflect * battery_dist / 2}
-                   0"
-              rpy="${reflect * battery_comp_angle} 0 0"/>
-    </joint>
-    <link name="${prefix}_battery_offset">
-      <xacro:null_inertial/>
-    </link>
-    <joint name="offset_to_${prefix}_battery" type="fixed">
-      <parent link="${prefix}_battery_offset"/>
-      <child link="${prefix}_battery"/>
-      <origin xyz="0
-                   ${reflect * battery_width / 2}
-                   ${(battery_height / 2) - battery_comp_depth}"/>
-    </joint>
-    <link name="${prefix}_battery">
-      <visual>
-        <geometry>
-          <box size="${battery_length} ${battery_width} ${battery_height}"/>
-        </geometry>
-        <material name="battery_mat"/>
-      </visual>
-      <collision>
-        <geometry>
-          <box size="${battery_length} ${battery_width} ${battery_height}"/>
-        </geometry>
-      </collision>
-      <xacro:solid_cuboid_inertial
-         width="${battery_length}" depth="${battery_width}"
-         height="${battery_height}" mass="${battery_mass}">
-        <origin/>
-      </xacro:solid_cuboid_inertial>
-    </link>
-    <gazebo reference="${prefix}_battery">
-      <material>Gazebo/Blue</material>
-    </gazebo>
-  </xacro:macro>
   <!-- Shock absorber -->
   <xacro:macro name="shock"
@@ -342,7 +300,4 @@
     <child link="chassis"/>
   </joint>
-  <!-- Batteries -->
-  <xacro:battery prefix="left" reflect="1"/>
-  <xacro:battery prefix="right" reflect="-1"/>
   <!-- Wheels -->
   <xacro:front_wheel lr_prefix="left" fr_prefix="front"
