Commit message: Add files via upload

File: ackermann_vehicle_description/urdf/archives/em_3905.urdf_V1.xacro (robot description, xacro)
@@ -1,3 +1,4 @@
 <?xml version="1.0"?>
+<!-- MADE SOME CHANGES IN THE DIMENSIONS -->
 <!-- em_3905.urdf.xacro
 This file defines a model of a Traxxas(R) E-Maxx(R) #3905 RC (Radio Controlled)
@@ -28,8 +29,4 @@
 -->
 <robot name="em_3905" xmlns:xacro="http://www.ros.org/wiki/xacro">
-  <xacro:include filename="$(find ackermann_vehicle_description)/urdf/colors.xacro" />
-  <xacro:include filename="$(find ackermann_vehicle_description)/urdf/sensors.gazebo" />
-  <xacro:property name="cameraSize" value="0.05"/>
-  <xacro:property name="cameraMass" value="0.1"/>
   <!-- Degree-to-radian conversions -->
   <xacro:property name="degrees_45" value="0.785398163"/>
@@ -37,8 +34,20 @@
   <!-- chassis_length is measured along the x axis, chassis_width
        along the y axis, and chassis_height along the z axis. -->
-  <xacro:property name="chassis_length" value="0.258"/>
-  <xacro:property name="chassis_width" value="0.168"/>
+  <xacro:property name="chassis_length" value="3.280"/>
+  <xacro:property name="chassis_width" value="1.514"/>
   <xacro:property name="chassis_height" value="0.01"/>
   <xacro:property name="chassis_mass" value="2.788"/>
+  <!-- battery_dist is the distance between the inner edges of the
+       batteries. battery_comp_depth is the battery compartment depth.
+       battery_length is measured along the x axis, battery_width
+       along the y axis, and battery_height along the z axis. -->
+  <xacro:property name="battery_x_offset" value="0.055"/>
+  <xacro:property name="battery_dist" value="0.065"/>
+  <xacro:property name="battery_comp_depth" value="0.02"/>
+  <xacro:property name="battery_comp_angle" value="0.34906585"/>
+  <xacro:property name="battery_length" value="0.16"/>
+  <xacro:property name="battery_width" value="0.047"/>
+  <xacro:property name="battery_height" value="0.024"/>
+  <xacro:property name="battery_mass" value="0.5025"/>
   <!-- hub_dia and tire_dia are the diameters of the hub and tire,
        respectively. hex_hub_depth is the distance that the hex hub is
@@ -47,5 +56,5 @@
        axle_length. -->
   <xacro:property name="hub_dia" value="0.09652"/>
-  <xacro:property name="tire_dia" value="0.14605"/>
+  <xacro:property name="tire_dia" value="0.3305"/>
   <xacro:property name="tire_width" value="0.0889"/>
   <xacro:property name="hex_hub_depth" value="0.01445"/>
@@ -55,6 +64,6 @@
        from a U joint to the corresponding hex hub. wheel_travel is the
        vertical wheel travel. -->
-  <xacro:property name="wheelbase" value="0.335"/>
-  <xacro:property name="hex_hub_dist" value="0.365"/>
+  <xacro:property name="wheelbase" value="1.958"/>
+  <xacro:property name="hex_hub_dist" value="1.2365"/>
   <xacro:property name="axle_length" value="0.03"/>
   <xacro:property name="wheel_travel" value="0.084"/>
@@ -83,6 +92,15 @@
        6 V. servo_stall_torque is measured in N m. servo_no_load_speed is
        measured in rad/s. -->
-  <xacro:property name="servo_stall_torque" value="0.5649"/>
-  <xacro:property name="servo_no_load_speed" value="4.553"/>
+  <xacro:property name="servo_stall_torque" value="1.5649"/>
+  <xacro:property name="servo_no_load_speed" value="4.5530"/>
+  <material name="battery_mat">
+    <color rgba="0 0 1 1"/>
+  </material>
+  <material name="chassis_mat">
+    <color rgba="0.5 0.5 0.5 1"/>
+  </material>
+  <material name="tire_mat">
+    <color rgba="0 0 0 1"/>
+  </material>
   <!-- Null inertial element. This is needed to make the model work with
        Gazebo. -->
@@ -123,4 +141,46 @@
                     outer_rad * outer_rad) / 2}"/>
     </inertial>
+  </xacro:macro>
+  <!-- Battery -->
+  <xacro:macro name="battery" params="prefix reflect">
+    <joint name="chassis_to_${prefix}_battery" type="fixed">
+      <parent link="chassis"/>
+      <child link="${prefix}_battery_offset"/>
+      <origin xyz="${battery_x_offset - battery_length / 2}
+                   ${reflect * battery_dist / 2}
+                   0"
+              rpy="${reflect * battery_comp_angle} 0 0"/>
+    </joint>
+    <link name="${prefix}_battery_offset">
+      <xacro:null_inertial/>
+    </link>
+    <joint name="offset_to_${prefix}_battery" type="fixed">
+      <parent link="${prefix}_battery_offset"/>
+      <child link="${prefix}_battery"/>
+      <origin xyz="0
+                   ${reflect * battery_width / 2}
+                   ${(battery_height / 2) - battery_comp_depth}"/>
+    </joint>
+    <link name="${prefix}_battery">
+      <visual>
+        <geometry>
+          <box size="${battery_length} ${battery_width} ${battery_height}"/>
+        </geometry>
+        <material name="battery_mat"/>
+      </visual>
+      <collision>
+        <geometry>
+          <box size="${battery_length} ${battery_width} ${battery_height}"/>
+        </geometry>
+      </collision>
+      <xacro:solid_cuboid_inertial
+         width="${battery_length}" depth="${battery_width}"
+         height="${battery_height}" mass="${battery_mass}">
+        <origin/>
+      </xacro:solid_cuboid_inertial>
+    </link>
+    <gazebo reference="${prefix}_battery">
+      <material>Gazebo/Blue</material>
+    </gazebo>
   </xacro:macro>
   <!-- Shock absorber -->
@@ -285,4 +345,7 @@
     <child link="chassis"/>
   </joint>
+  <!-- Batteries -->
+  <xacro:battery prefix="left" reflect="1"/>
+  <xacro:battery prefix="right" reflect="-1"/>
   <!-- Wheels -->
   <xacro:front_wheel lr_prefix="left" fr_prefix="front"
@@ -294,85 +357,4 @@
   <xacro:rear_wheel lr_prefix="right" fr_prefix="rear"
                     lr_reflect="-1" fr_reflect="-1"/>
-  <link name="camera">
-    <collision>
-      <origin xyz="0 0 0" rpy="0 0 0"/>
-      <geometry>
-        <box size="${cameraSize} ${cameraSize} ${cameraSize}"/>
-      </geometry>
-    </collision>
-    <visual>
-      <origin xyz="0 0 0" rpy="0 0 0"/>
-      <geometry>
-        <box size="${cameraSize} ${cameraSize} ${cameraSize}"/>
-      </geometry>
-      <material name="battery_mat"/>
-    </visual>
-    <inertial>
-      <mass value="${cameraMass}" />
-      <origin xyz="0 0 0" rpy="0 0 0"/>
-      <box_inertia m="${cameraMass}" x="${cameraSize}" y="${cameraSize}" z="${cameraSize}" />
-      <inertia ixx="1e-6" ixy="0" ixz="0" iyy="1e-6" iyz="0" izz="1e-6" />
-    </inertial>
-  </link>
-  <joint name="camera_joint" type="fixed">
-    <axis xyz="0 1 0" />
-    <origin xyz=".2 0 1" rpy="0 0 0"/>
-    <parent link="chassis"/>
-    <child link="camera"/>
-  </joint>
-  <link name="left_camera_frame">
-    <collision>
-      <origin xyz="0 0 0" rpy="0 0 0"/>
-      <geometry>
-        <box size="${cameraSize} ${cameraSize} ${cameraSize}"/>
-      </geometry>
-    </collision>
-    <visual>
-      <origin xyz="0 0 0" rpy="0 0 0"/>
-      <geometry>
-        <box size="${cameraSize} ${cameraSize} ${cameraSize}"/>
-      </geometry>
-      <material name="chassis_mat"/>
-    </visual>
-    <inertial>
-      <mass value="${cameraMass}" />
-      <origin xyz="0 0 0" rpy="0 0 0"/>
-      <box_inertia m="${cameraMass}" x="${cameraSize}" y="${cameraSize}" z="${cameraSize}" />
-      <inertia ixx="1e-6" ixy="0" ixz="0" iyy="1e-6" iyz="0" izz="1e-6" />
-    </inertial>
-  </link>
-  <joint name="stereo_camera_joint" type="fixed">
-    <axis xyz="0 1 0" />
-    <origin xyz=".2 0 0.7" rpy="0 0 0"/>
-    <parent link="chassis"/>
-    <child link="left_camera_frame"/>
-  </joint>
-  <link name="imu_link">
-    <collision>
-      <origin xyz="0 0 0" rpy="0 0 0"/>
-      <geometry>
-        <box size="${cameraSize} ${cameraSize} ${cameraSize}"/>
-      </geometry>
-    </collision>
-    <visual>
-      <origin xyz="0 0 0" rpy="0 0 0"/>
-      <geometry>
-        <box size="${cameraSize} ${cameraSize} ${cameraSize}"/>
-      </geometry>
-      <material name="blue"/>
-    </visual>
-    <inertial>
-      <mass value="${cameraMass}" />
-      <origin xyz="0 0 0" rpy="0 0 0"/>
-      <box_inertia m="${cameraMass}" x="${cameraSize}" y="${cameraSize}" z="${cameraSize}" />
-      <inertia ixx="1e-6" ixy="0" ixz="0" iyy="1e-6" iyz="0" izz="1e-6" />
-    </inertial>
-  </link>
-  <joint name="imu_joint" type="fixed">
-    <axis xyz="0 1 0" />
-    <origin xyz=".2 0 0.5" rpy="0 0 0"/>
-    <parent link="chassis"/>
-    <child link="imu_link"/>
-  </joint>
   <gazebo>
     <plugin name="gazebo_ros_control" filename="libgazebo_ros_control.so"/>

File: ackermann_vehicle_description/urdf/archives/em_3905.urdf_V2.xacro (robot description, xacro)
@@ -1,3 +1,6 @@
 <?xml version="1.0"?>
+<!-- MADE SOME CHANGES IN THE DIMENSIONS and MASS
+WHEEL MASS IS CORRECT, REST IS NOT -->
+<!-- rEMOVED THE BATTERIES -->
 <!-- em_3905.urdf.xacro
 This file defines a model of a Traxxas(R) E-Maxx(R) #3905 RC (Radio Controlled)
@@ -29,7 +32,4 @@
 <robot name="em_3905" xmlns:xacro="http://www.ros.org/wiki/xacro">
   <xacro:include filename="$(find ackermann_vehicle_description)/urdf/colors.xacro" />
-  <xacro:include filename="$(find ackermann_vehicle_description)/urdf/sensors.gazebo" />
-  <xacro:property name="cameraSize" value="0.05"/>
-  <xacro:property name="cameraMass" value="0.1"/>
   <!-- Degree-to-radian conversions -->
   <xacro:property name="degrees_45" value="0.785398163"/>
@@ -37,8 +37,8 @@
   <!-- chassis_length is measured along the x axis, chassis_width
        along the y axis, and chassis_height along the z axis. -->
-  <xacro:property name="chassis_length" value="0.258"/>
-  <xacro:property name="chassis_width" value="0.168"/>
+  <xacro:property name="chassis_length" value="3.280"/>
+  <xacro:property name="chassis_width" value="1.514"/>
   <xacro:property name="chassis_height" value="0.01"/>
-  <xacro:property name="chassis_mass" value="2.788"/>
+  <xacro:property name="chassis_mass" value="40.788"/>
   <!-- hub_dia and tire_dia are the diameters of the hub and tire,
        respectively. hex_hub_depth is the distance that the hex hub is
@@ -47,22 +47,22 @@
        axle_length. -->
   <xacro:property name="hub_dia" value="0.09652"/>
-  <xacro:property name="tire_dia" value="0.14605"/>
+  <xacro:property name="tire_dia" value="0.3305"/>
   <xacro:property name="tire_width" value="0.0889"/>
   <xacro:property name="hex_hub_depth" value="0.01445"/>
-  <xacro:property name="wheel_mass" value="0.29"/>
+  <xacro:property name="wheel_mass" value="8.00"/>
   <!-- hex_hub_dist is the distance between left and right hex hubs when
        the shock absorbers are fully extended. axle_length is the distance
        from a U joint to the corresponding hex hub. wheel_travel is the
        vertical wheel travel. -->
-  <xacro:property name="wheelbase" value="0.335"/>
-  <xacro:property name="hex_hub_dist" value="0.365"/>
+  <xacro:property name="wheelbase" value="1.958"/>
+  <xacro:property name="hex_hub_dist" value="1.2365"/>
   <xacro:property name="axle_length" value="0.03"/>
   <xacro:property name="wheel_travel" value="0.084"/>
-  <xacro:property name="shock_z_offset" value="0.0655"/>
+  <xacro:property name="shock_z_offset" value="0.1"/> <!-- Set the value to 0.255 after you solve the wheel problem-->
   <!-- shock_eff_limit is 2 * ((shock_stroke / 2) * shock_spring_constant) N.
        shock_stroke is 0.028575 meters. shock_spring_constant, an approximation
        of a Traxxas Ultra Shock shock absorber spring's constant, is
        437.817 N/m. -->
-  <xacro:property name="shock_eff_limit" value="12.5106"/>
+  <xacro:property name="shock_eff_limit" value="1000.5106"/>
   <xacro:property name="shock_vel_limit" value="1000"/>
   <!-- The specifications for a Titan(R) 550 motor could not be found, so the
@@ -79,10 +79,10 @@
          244.8696 rad/s -->
   <xacro:property name="axle_eff_limit" value="5.12766"/>
-  <xacro:property name="axle_vel_limit" value="244.8696"/>
+  <xacro:property name="axle_vel_limit" value="50.8696"/>
   <!-- These constants are used to simulate a Traxxas 2056 servo operated at
        6 V. servo_stall_torque is measured in N m. servo_no_load_speed is
        measured in rad/s. -->
-  <xacro:property name="servo_stall_torque" value="0.5649"/>
-  <xacro:property name="servo_no_load_speed" value="4.553"/>
+  <xacro:property name="servo_stall_torque" value="1.5649"/>
+  <xacro:property name="servo_no_load_speed" value="4.5530"/>
   <!-- Null inertial element. This is needed to make the model work with
        Gazebo. -->
@@ -294,85 +294,4 @@
   <xacro:rear_wheel lr_prefix="right" fr_prefix="rear"
                     lr_reflect="-1" fr_reflect="-1"/>
-  <link name="camera">
-    <collision>
-      <origin xyz="0 0 0" rpy="0 0 0"/>
-      <geometry>
-        <box size="${cameraSize} ${cameraSize} ${cameraSize}"/>
-      </geometry>
-    </collision>
-    <visual>
-      <origin xyz="0 0 0" rpy="0 0 0"/>
-      <geometry>
-        <box size="${cameraSize} ${cameraSize} ${cameraSize}"/>
-      </geometry>
-      <material name="battery_mat"/>
-    </visual>
-    <inertial>
-      <mass value="${cameraMass}" />
-      <origin xyz="0 0 0" rpy="0 0 0"/>
-      <box_inertia m="${cameraMass}" x="${cameraSize}" y="${cameraSize}" z="${cameraSize}" />
-      <inertia ixx="1e-6" ixy="0" ixz="0" iyy="1e-6" iyz="0" izz="1e-6" />
-    </inertial>
-  </link>
-  <joint name="camera_joint" type="fixed">
-    <axis xyz="0 1 0" />
-    <origin xyz=".2 0 1" rpy="0 0 0"/>
-    <parent link="chassis"/>
-    <child link="camera"/>
-  </joint>
-  <link name="left_camera_frame">
-    <collision>
-      <origin xyz="0 0 0" rpy="0 0 0"/>
-      <geometry>
-        <box size="${cameraSize} ${cameraSize} ${cameraSize}"/>
-      </geometry>
-    </collision>
-    <visual>
-      <origin xyz="0 0 0" rpy="0 0 0"/>
-      <geometry>
-        <box size="${cameraSize} ${cameraSize} ${cameraSize}"/>
-      </geometry>
-      <material name="chassis_mat"/>
-    </visual>
-    <inertial>
-      <mass value="${cameraMass}" />
-      <origin xyz="0 0 0" rpy="0 0 0"/>
-      <box_inertia m="${cameraMass}" x="${cameraSize}" y="${cameraSize}" z="${cameraSize}" />
-      <inertia ixx="1e-6" ixy="0" ixz="0" iyy="1e-6" iyz="0" izz="1e-6" />
-    </inertial>
-  </link>
-  <joint name="stereo_camera_joint" type="fixed">
-    <axis xyz="0 1 0" />
-    <origin xyz=".2 0 0.7" rpy="0 0 0"/>
-    <parent link="chassis"/>
-    <child link="left_camera_frame"/>
-  </joint>
-  <link name="imu_link">
-    <collision>
-      <origin xyz="0 0 0" rpy="0 0 0"/>
-      <geometry>
-        <box size="${cameraSize} ${cameraSize} ${cameraSize}"/>
-      </geometry>
-    </collision>
-    <visual>
-      <origin xyz="0 0 0" rpy="0 0 0"/>
-      <geometry>
-        <box size="${cameraSize} ${cameraSize} ${cameraSize}"/>
-      </geometry>
-      <material name="blue"/>
-    </visual>
-    <inertial>
-      <mass value="${cameraMass}" />
-      <origin xyz="0 0 0" rpy="0 0 0"/>
-      <box_inertia m="${cameraMass}" x="${cameraSize}" y="${cameraSize}" z="${cameraSize}" />
-      <inertia ixx="1e-6" ixy="0" ixz="0" iyy="1e-6" iyz="0" izz="1e-6" />
-    </inertial>
-  </link>
-  <joint name="imu_joint" type="fixed">
-    <axis xyz="0 1 0" />
-    <origin xyz=".2 0 0.5" rpy="0 0 0"/>
-    <parent link="chassis"/>
-    <child link="imu_link"/>
-  </joint>
   <gazebo>
     <plugin name="gazebo_ros_control" filename="libgazebo_ros_control.so"/>

File: ackermann_vehicle_description/urdf/archives/em_3905.urdf_V3.xacro (robot description, xacro)
@@ -1,3 +1,6 @@
 <?xml version="1.0"?>
+<!-- MADE CHANGES IN THE DIMENSIONS and MASS
+WHEEL MASS IS CORRECT, REST IS NOT -->
+<!-- Also added a camera, imu and broke the materials to a different file -->
 <!-- em_3905.urdf.xacro
 This file defines a model of a Traxxas(R) E-Maxx(R) #3905 RC (Radio Controlled)
@@ -37,8 +40,20 @@
   <!-- chassis_length is measured along the x axis, chassis_width
        along the y axis, and chassis_height along the z axis. -->
-  <xacro:property name="chassis_length" value="0.258"/>
-  <xacro:property name="chassis_width" value="0.168"/>
+  <xacro:property name="chassis_length" value="3.280"/>
+  <xacro:property name="chassis_width" value="1.514"/>
   <xacro:property name="chassis_height" value="0.01"/>
   <xacro:property name="chassis_mass" value="2.788"/>
+  <!-- battery_dist is the distance between the inner edges of the
+       batteries. battery_comp_depth is the battery compartment depth.
+       battery_length is measured along the x axis, battery_width
+       along the y axis, and battery_height along the z axis. -->
+  <xacro:property name="battery_x_offset" value="0.055"/>
+  <xacro:property name="battery_dist" value="0.065"/>
+  <xacro:property name="battery_comp_depth" value="0.02"/>
+  <xacro:property name="battery_comp_angle" value="0.34906585"/>
+  <xacro:property name="battery_length" value="0.16"/>
+  <xacro:property name="battery_width" value="0.047"/>
+  <xacro:property name="battery_height" value="0.024"/>
+  <xacro:property name="battery_mass" value="0.5025"/>
   <!-- hub_dia and tire_dia are the diameters of the hub and tire,
        respectively. hex_hub_depth is the distance that the hex hub is
@@ -47,14 +62,14 @@
        axle_length. -->
   <xacro:property name="hub_dia" value="0.09652"/>
-  <xacro:property name="tire_dia" value="0.14605"/>
+  <xacro:property name="tire_dia" value="0.3305"/>
   <xacro:property name="tire_width" value="0.0889"/>
   <xacro:property name="hex_hub_depth" value="0.01445"/>
-  <xacro:property name="wheel_mass" value="0.29"/>
+  <xacro:property name="wheel_mass" value="8.00"/>
   <!-- hex_hub_dist is the distance between left and right hex hubs when
        the shock absorbers are fully extended. axle_length is the distance
        from a U joint to the corresponding hex hub. wheel_travel is the
        vertical wheel travel. -->
-  <xacro:property name="wheelbase" value="0.335"/>
-  <xacro:property name="hex_hub_dist" value="0.365"/>
+  <xacro:property name="wheelbase" value="1.958"/>
+  <xacro:property name="hex_hub_dist" value="1.2365"/>
   <xacro:property name="axle_length" value="0.03"/>
   <xacro:property name="wheel_travel" value="0.084"/>
@@ -83,6 +98,6 @@
        6 V. servo_stall_torque is measured in N m. servo_no_load_speed is
        measured in rad/s. -->
-  <xacro:property name="servo_stall_torque" value="0.5649"/>
-  <xacro:property name="servo_no_load_speed" value="4.553"/>
+  <xacro:property name="servo_stall_torque" value="1.5649"/>
+  <xacro:property name="servo_no_load_speed" value="4.5530"/>
   <!-- Null inertial element. This is needed to make the model work with
        Gazebo. -->
@@ -123,4 +138,46 @@
                     outer_rad * outer_rad) / 2}"/>
     </inertial>
+  </xacro:macro>
+  <!-- Battery -->
+  <xacro:macro name="battery" params="prefix reflect">
+    <joint name="chassis_to_${prefix}_battery" type="fixed">
+      <parent link="chassis"/>
+      <child link="${prefix}_battery_offset"/>
+      <origin xyz="${battery_x_offset - battery_length / 2}
+                   ${reflect * battery_dist / 2}
+                   0"
+              rpy="${reflect * battery_comp_angle} 0 0"/>
+    </joint>
+    <link name="${prefix}_battery_offset">
+      <xacro:null_inertial/>
+    </link>
+    <joint name="offset_to_${prefix}_battery" type="fixed">
+      <parent link="${prefix}_battery_offset"/>
+      <child link="${prefix}_battery"/>
+      <origin xyz="0
+                   ${reflect * battery_width / 2}
+                   ${(battery_height / 2) - battery_comp_depth}"/>
+    </joint>
+    <link name="${prefix}_battery">
+      <visual>
+        <geometry>
+          <box size="${battery_length} ${battery_width} ${battery_height}"/>
+        </geometry>
+        <material name="battery_mat"/>
+      </visual>
+      <collision>
+        <geometry>
+          <box size="${battery_length} ${battery_width} ${battery_height}"/>
+        </geometry>
+      </collision>
+      <xacro:solid_cuboid_inertial
+         width="${battery_length}" depth="${battery_width}"
+         height="${battery_height}" mass="${battery_mass}">
+        <origin/>
+      </xacro:solid_cuboid_inertial>
+    </link>
+    <gazebo reference="${prefix}_battery">
+      <material>Gazebo/Blue</material>
+    </gazebo>
   </xacro:macro>
   <!-- Shock absorber -->
@@ -285,4 +342,7 @@
     <child link="chassis"/>
   </joint>
+  <!-- Batteries -->
+  <xacro:battery prefix="left" reflect="1"/>
+  <xacro:battery prefix="right" reflect="-1"/>
   <!-- Wheels -->
   <xacro:front_wheel lr_prefix="left" fr_prefix="front"
@@ -306,5 +366,5 @@
         <box size="${cameraSize} ${cameraSize} ${cameraSize}"/>
       </geometry>
-      <material name="battery_mat"/>
+      <material name="green"/>
     </visual>
     <inertial>
@@ -320,31 +380,4 @@
     <parent link="chassis"/>
     <child link="camera"/>
-  </joint>
-  <link name="left_camera_frame">
-    <collision>
-      <origin xyz="0 0 0" rpy="0 0 0"/>
-      <geometry>
-        <box size="${cameraSize} ${cameraSize} ${cameraSize}"/>
-      </geometry>
-    </collision>
-    <visual>
-      <origin xyz="0 0 0" rpy="0 0 0"/>
-      <geometry>
-        <box size="${cameraSize} ${cameraSize} ${cameraSize}"/>
-      </geometry>
-      <material name="chassis_mat"/>
-    </visual>
-    <inertial>
-      <mass value="${cameraMass}" />
-      <origin xyz="0 0 0" rpy="0 0 0"/>
-      <box_inertia m="${cameraMass}" x="${cameraSize}" y="${cameraSize}" z="${cameraSize}" />
-      <inertia ixx="1e-6" ixy="0" ixz="0" iyy="1e-6" iyz="0" izz="1e-6" />
-    </inertial>
-  </link>
-  <joint name="stereo_camera_joint" type="fixed">
-    <axis xyz="0 1 0" />
-    <origin xyz=".2 0 0.7" rpy="0 0 0"/>
-    <parent link="chassis"/>
-    <child link="left_camera_frame"/>
   </joint>
   <link name="imu_link">
