Commit message: Add files via upload

File: ackermann_vehicle_description/urdf/archives/em_3905.urdf_V4.xacro (robot description, xacro)
@@ -1,3 +1,6 @@
 <?xml version="1.0"?>
+<!-- MADE SOME CHANGES IN THE DIMENSIONS and MASS
+WHEEL MASS IS CORRECT, REST IS NOT -->
+<!-- Also added a camera, imu, removed the batteries and broke the materials to a different file -->
 <!-- em_3905.urdf.xacro
 This file defines a model of a Traxxas(R) E-Maxx(R) #3905 RC (Radio Controlled)
@@ -37,8 +40,20 @@
   <!-- chassis_length is measured along the x axis, chassis_width
        along the y axis, and chassis_height along the z axis. -->
-  <xacro:property name="chassis_length" value="0.258"/>
-  <xacro:property name="chassis_width" value="0.168"/>
+  <xacro:property name="chassis_length" value="3.280"/>
+  <xacro:property name="chassis_width" value="1.514"/>
   <xacro:property name="chassis_height" value="0.01"/>
   <xacro:property name="chassis_mass" value="2.788"/>
+  <!-- battery_dist is the distance between the inner edges of the
+       batteries. battery_comp_depth is the battery compartment depth.
+       battery_length is measured along the x axis, battery_width
+       along the y axis, and battery_height along the z axis. -->
+  <xacro:property name="battery_x_offset" value="0.055"/>
+  <xacro:property name="battery_dist" value="0.065"/>
+  <xacro:property name="battery_comp_depth" value="0.02"/>
+  <xacro:property name="battery_comp_angle" value="0.34906585"/>
+  <xacro:property name="battery_length" value="0.16"/>
+  <xacro:property name="battery_width" value="0.047"/>
+  <xacro:property name="battery_height" value="0.024"/>
+  <xacro:property name="battery_mass" value="0.5025"/>
   <!-- hub_dia and tire_dia are the diameters of the hub and tire,
        respectively. hex_hub_depth is the distance that the hex hub is
@@ -47,14 +62,14 @@
        axle_length. -->
   <xacro:property name="hub_dia" value="0.09652"/>
-  <xacro:property name="tire_dia" value="0.14605"/>
+  <xacro:property name="tire_dia" value="0.3305"/>
   <xacro:property name="tire_width" value="0.0889"/>
   <xacro:property name="hex_hub_depth" value="0.01445"/>
-  <xacro:property name="wheel_mass" value="0.29"/>
+  <xacro:property name="wheel_mass" value="8.00"/>
   <!-- hex_hub_dist is the distance between left and right hex hubs when
        the shock absorbers are fully extended. axle_length is the distance
        from a U joint to the corresponding hex hub. wheel_travel is the
        vertical wheel travel. -->
-  <xacro:property name="wheelbase" value="0.335"/>
-  <xacro:property name="hex_hub_dist" value="0.365"/>
+  <xacro:property name="wheelbase" value="1.958"/>
+  <xacro:property name="hex_hub_dist" value="1.2365"/>
   <xacro:property name="axle_length" value="0.03"/>
   <xacro:property name="wheel_travel" value="0.084"/>
@@ -83,6 +98,6 @@
        6 V. servo_stall_torque is measured in N m. servo_no_load_speed is
        measured in rad/s. -->
-  <xacro:property name="servo_stall_torque" value="0.5649"/>
-  <xacro:property name="servo_no_load_speed" value="4.553"/>
+  <xacro:property name="servo_stall_torque" value="1.5649"/>
+  <xacro:property name="servo_no_load_speed" value="4.5530"/>
   <!-- Null inertial element. This is needed to make the model work with
        Gazebo. -->
@@ -306,5 +321,5 @@
         <box size="${cameraSize} ${cameraSize} ${cameraSize}"/>
       </geometry>
-      <material name="battery_mat"/>
+      <material name="green"/>
     </visual>
     <inertial>
@@ -320,31 +335,4 @@
     <parent link="chassis"/>
     <child link="camera"/>
-  </joint>
-  <link name="left_camera_frame">
-    <collision>
-      <origin xyz="0 0 0" rpy="0 0 0"/>
-      <geometry>
-        <box size="${cameraSize} ${cameraSize} ${cameraSize}"/>
-      </geometry>
-    </collision>
-    <visual>
-      <origin xyz="0 0 0" rpy="0 0 0"/>
-      <geometry>
-        <box size="${cameraSize} ${cameraSize} ${cameraSize}"/>
-      </geometry>
-      <material name="chassis_mat"/>
-    </visual>
-    <inertial>
-      <mass value="${cameraMass}" />
-      <origin xyz="0 0 0" rpy="0 0 0"/>
-      <box_inertia m="${cameraMass}" x="${cameraSize}" y="${cameraSize}" z="${cameraSize}" />
-      <inertia ixx="1e-6" ixy="0" ixz="0" iyy="1e-6" iyz="0" izz="1e-6" />
-    </inertial>
-  </link>
-  <joint name="stereo_camera_joint" type="fixed">
-    <axis xyz="0 1 0" />
-    <origin xyz=".2 0 0.7" rpy="0 0 0"/>
-    <parent link="chassis"/>
-    <child link="left_camera_frame"/>
   </joint>
   <link name="imu_link">

File: ackermann_vehicle_description/urdf/archives/em_3905.urdf_V5.xacro (robot description, xacro)
@@ -1,3 +1,7 @@
 <?xml version="1.0"?>
+<!-- MADE SOME CHANGES IN THE DIMENSIONS and MASS
+WHEEL MASS IS CORRECT, REST IS NOT -->
+<!-- Also added a camera, imu, removed the batteries and broke the materials to a different file -->
+<!-- ADDed a stereo camera -->
 <!-- em_3905.urdf.xacro
 This file defines a model of a Traxxas(R) E-Maxx(R) #3905 RC (Radio Controlled)
@@ -37,6 +41,6 @@
   <!-- chassis_length is measured along the x axis, chassis_width
        along the y axis, and chassis_height along the z axis. -->
-  <xacro:property name="chassis_length" value="0.258"/>
-  <xacro:property name="chassis_width" value="0.168"/>
+  <xacro:property name="chassis_length" value="3.280"/>
+  <xacro:property name="chassis_width" value="1.514"/>
   <xacro:property name="chassis_height" value="0.01"/>
   <xacro:property name="chassis_mass" value="2.788"/>
@@ -47,14 +51,14 @@
        axle_length. -->
   <xacro:property name="hub_dia" value="0.09652"/>
-  <xacro:property name="tire_dia" value="0.14605"/>
-  <xacro:property name="tire_width" value="0.0889"/>
+  <xacro:property name="tire_dia" value="0.3305"/>
+  <xacro:property name="tire_width" value="0.155"/>
   <xacro:property name="hex_hub_depth" value="0.01445"/>
-  <xacro:property name="wheel_mass" value="0.29"/>
+  <xacro:property name="wheel_mass" value="8.00"/>
   <!-- hex_hub_dist is the distance between left and right hex hubs when
        the shock absorbers are fully extended. axle_length is the distance
        from a U joint to the corresponding hex hub. wheel_travel is the
        vertical wheel travel. -->
-  <xacro:property name="wheelbase" value="0.335"/>
-  <xacro:property name="hex_hub_dist" value="0.365"/>
+  <xacro:property name="wheelbase" value="1.958"/>
+  <xacro:property name="hex_hub_dist" value="1.2365"/>
   <xacro:property name="axle_length" value="0.03"/>
   <xacro:property name="wheel_travel" value="0.084"/>
@@ -83,6 +87,6 @@
        6 V. servo_stall_torque is measured in N m. servo_no_load_speed is
        measured in rad/s. -->
-  <xacro:property name="servo_stall_torque" value="0.5649"/>
-  <xacro:property name="servo_no_load_speed" value="4.553"/>
+  <xacro:property name="servo_stall_torque" value="1.5649"/>
+  <xacro:property name="servo_no_load_speed" value="4.5530"/>
   <!-- Null inertial element. This is needed to make the model work with
        Gazebo. -->

File: ackermann_vehicle_description/urdf/colors.xacro (robot description, xacro)
@@ -2,5 +2,5 @@
 <robot>
   <material name="blue">
-    <color rgba="0.0 0.0 0.8 1.0"/>
+    <color rgba="0.0 0.0 0.5 1.0"/>
   </material>
   <material name="green">

File: ackermann_vehicle_description/urdf/em_3905.urdf_VV1.xacro (robot description, xacro)
@@ -37,6 +37,6 @@
   <!-- chassis_length is measured along the x axis, chassis_width
        along the y axis, and chassis_height along the z axis. -->
-  <xacro:property name="chassis_length" value="0.258"/>
-  <xacro:property name="chassis_width" value="0.168"/>
+  <xacro:property name="chassis_length" value="3.280"/> <!-- SET -->
+  <xacro:property name="chassis_width" value="1.514"/> <!-- SET -->
   <xacro:property name="chassis_height" value="0.01"/>
   <xacro:property name="chassis_mass" value="2.788"/>
@@ -47,17 +47,17 @@
        axle_length. -->
   <xacro:property name="hub_dia" value="0.09652"/>
-  <xacro:property name="tire_dia" value="0.14605"/>
+  <xacro:property name="tire_dia" value="0.33"/> <!-- SET -->
   <xacro:property name="tire_width" value="0.0889"/>
   <xacro:property name="hex_hub_depth" value="0.01445"/>
-  <xacro:property name="wheel_mass" value="0.29"/>
+  <xacro:property name="wheel_mass" value="8.0"/>
   <!-- hex_hub_dist is the distance between left and right hex hubs when
        the shock absorbers are fully extended. axle_length is the distance
        from a U joint to the corresponding hex hub. wheel_travel is the
        vertical wheel travel. -->
-  <xacro:property name="wheelbase" value="0.335"/>
-  <xacro:property name="hex_hub_dist" value="0.365"/>
+  <xacro:property name="wheelbase" value="1.958"/>  <!-- SET -->
+  <xacro:property name="hex_hub_dist" value="1.20"/>
   <xacro:property name="axle_length" value="0.03"/>
   <xacro:property name="wheel_travel" value="0.084"/>
-  <xacro:property name="shock_z_offset" value="0.0655"/>
+  <xacro:property name="shock_z_offset" value="0.25"/> <!-- SET -->
   <!-- shock_eff_limit is 2 * ((shock_stroke / 2) * shock_spring_constant) N.
        shock_stroke is 0.028575 meters. shock_spring_constant, an approximation
@@ -83,5 +83,5 @@
        6 V. servo_stall_torque is measured in N m. servo_no_load_speed is
        measured in rad/s. -->
-  <xacro:property name="servo_stall_torque" value="0.5649"/>
+  <xacro:property name="servo_stall_torque" value="1.5649"/>
   <xacro:property name="servo_no_load_speed" value="4.553"/>
   <!-- Null inertial element. This is needed to make the model work with

File: ackermann_vehicle_description/urdf/model_test.xacro (robot description, xacro)
@@ -1,4 +1,5 @@
 <?xml version="1.0"?>
-<!-- em_3905.urdf.xacro
+<!-- em_3905.urdf.xacro -->
+<!-- ADDED THE CAR MODEL
 This file defines a model of a Traxxas(R) E-Maxx(R) #3905 RC (Radio Controlled)
 truck.
@@ -30,4 +31,5 @@
   <xacro:include filename="$(find ackermann_vehicle_description)/urdf/colors.xacro" />
   <xacro:include filename="$(find ackermann_vehicle_description)/urdf/sensors.gazebo" />
+  <xacro:include filename="$(find ackermann_vehicle_description)/urdf/e2o_without_tires.dae" />
   <xacro:property name="cameraSize" value="0.05"/>
   <xacro:property name="cameraMass" value="0.1"/>
@@ -37,6 +39,6 @@
   <!-- chassis_length is measured along the x axis, chassis_width
        along the y axis, and chassis_height along the z axis. -->
-  <xacro:property name="chassis_length" value="0.258"/>
-  <xacro:property name="chassis_width" value="0.168"/>
+  <xacro:property name="chassis_length" value="2.8"/> <!-- SET -->
+  <xacro:property name="chassis_width" value="1.2"/> <!-- SET -->
   <xacro:property name="chassis_height" value="0.01"/>
   <xacro:property name="chassis_mass" value="2.788"/>
@@ -47,17 +49,17 @@
        axle_length. -->
   <xacro:property name="hub_dia" value="0.09652"/>
-  <xacro:property name="tire_dia" value="0.14605"/>
+  <xacro:property name="tire_dia" value="0.5"/> <!-- SET -->
   <xacro:property name="tire_width" value="0.0889"/>
   <xacro:property name="hex_hub_depth" value="0.01445"/>
-  <xacro:property name="wheel_mass" value="0.29"/>
+  <xacro:property name="wheel_mass" value="8.0"/>
   <!-- hex_hub_dist is the distance between left and right hex hubs when
        the shock absorbers are fully extended. axle_length is the distance
        from a U joint to the corresponding hex hub. wheel_travel is the
        vertical wheel travel. -->
-  <xacro:property name="wheelbase" value="0.335"/>
-  <xacro:property name="hex_hub_dist" value="0.365"/>
+  <xacro:property name="wheelbase" value="1.958"/>  <!-- SET -->
+  <xacro:property name="hex_hub_dist" value="1.20"/>
   <xacro:property name="axle_length" value="0.03"/>
   <xacro:property name="wheel_travel" value="0.084"/>
-  <xacro:property name="shock_z_offset" value="0.0655"/>
+  <xacro:property name="shock_z_offset" value="0.25"/> <!-- SET -->
   <!-- shock_eff_limit is 2 * ((shock_stroke / 2) * shock_spring_constant) N.
        shock_stroke is 0.028575 meters. shock_spring_constant, an approximation
@@ -83,5 +85,5 @@
        6 V. servo_stall_torque is measured in N m. servo_no_load_speed is
        measured in rad/s. -->
-  <xacro:property name="servo_stall_torque" value="0.5649"/>
+  <xacro:property name="servo_stall_torque" value="1.5649"/>
   <xacro:property name="servo_no_load_speed" value="4.553"/>
   <!-- Null inertial element. This is needed to make the model work with
@@ -375,4 +377,18 @@
     <child link="imu_link"/>
   </joint>
+  <link name="car_model">
+        <visual name="visual">
+          <geometry>
+            <mesh filename="$(find ackermann_vehicle_description)/urdf/e2o_without_tires.dae"/>
+<!--	    <mesh><uri>file://e2o_without_tires.dae</uri></mesh> -->
+          </geometry>
+        </visual>
+  </link>
+  <joint name="car_joint" type="fixed">
+    <axis xyz="0 0 0" />
+    <origin xyz="1.5 0.95 -0.5" rpy="0 0 0"/>
+    <parent link="chassis"/>
+    <child link="car_model"/>
+  </joint>
   <gazebo>
     <plugin name="gazebo_ros_control" filename="libgazebo_ros_control.so"/>
